File: Mikadapter.kicad_sch (KiCad schematic)
At the start: 10 parts, among them J1 FC68131, J2 Conn_01x04_Female, J3 FC68131, J4 FC68131, J5 Conn_01x02_Female, J6 Conn_01x03_Female, J7 Conn_01x02_Female, J9 Conn_01x03_Female

Commit message: added schema as PDF and changed schema informations
Other:
- company: (none) -> DO7GN
- title: (none) -> Mikadpater FT81X
Changed lines of the file:
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@@
 (kicad_sch (version 20210621) (generator eeschema)
   (paper "A4")
+  (title_block
+    (title "Mikadpater FT81X")
+    (date "2021-09-30")
+    (rev "1.1")
+    (company "DO7GN")
+  )
   (global_label "MIC-" (shape input) (at 81.28 132.08 0) (fields_autoplaced)
     (effects (font (size 1.27 1.27)) (justify left))

Commit message: Changed Audio pins after inspection of the jack
Parts:
- removed J2: Conn_01x04_Female, Connector_PinHeader_2.54mm:PinHeader_1x04_P2.54mm_Vertical, symbol Connector:Conn_01x04_Female
- added J8: Conn_01x04_Female, Connector_PinHeader_2.54mm:PinHeader_2x03_P2.54mm_Vertical, symbol Connector_Generic:Conn_02x03_Odd_Even
Connections:
- net Audio+: now also J3.5, J4.5; no longer J3.2, J4.2
- net DWN: now also J8.5 (Pin_5)
- net FST: now also J8.3 (Pin_3)
- net GND: now also J8.2 (Pin_2), J8.4 (Pin_4), J8.6 (Pin_6)
- net MIC+: now also J1.5; no longer J1.2
- net UP: now also J8.1 (Pin_1)
