File: PCB/Mikadapter.kicad_pcb (KiCad board)
At the start: 2 copper layers, 57.1 x 50.8 mm, 18 parts, among them J1 FC68131, J3 FC68131, J4 FC68131, J5 Conn_01x02_Female, J6 Conn_01x03_Female, J7 Conn_01x02_Female, J8 Conn_01x04_Female, J9 Conn_01x03_Female

Commit message: Added trace for second Audio channel, new folder, 3D
Parts:
- added JP1: Jumper_2_Open, Jumper:SolderJumper-2_P1.3mm_Open_TrianglePad1.0x1.5mm, B.Cu at (156.5, 90.9)
Connections:
- J3 pad 1: Audio- -> AudioGND
- J3 pad 2: unconnected-(J3-Pad2) -> Audio-
- J4 pad 1: Audio- -> AudioGND
- J4 pad 2: unconnected-(J4-Pad2) -> Audio-
- J9 pad 1: Audio- -> AudioGND
Routing:
- net AudioGND: track 0.00 -> 59.3 mm
- net Audio+: track 57.7 -> 63.1 mm, vias 0 -> 1
- net Audio-: track 57.9 -> 53.4 mm, vias 0 -> 1
- net GND: vias 12 -> 15
